File: spartan6/hardware/dockerkit.brd (EAGLE design)
At the start: 85 x 56 mm, 6 parts

Commit message: 调整电路
Parts:
- removed U$6: DDR3, FPGA:FBGA96
- added R1: 240, Resistors&Capacitors:R0402
- added U$2: DDR3, IC_Memory:FBGA96
- U$4: device FPGA:FTG256 -> IC_FPGA:FTG256
Connections:
- removed net B0_G5: U$4.C7
- removed net B0_G6: U$4.A7
- removed net B0_G7: U$4.C9
- removed net B0_G8: U$4.A9
- removed net D2_N: U$4.A5
- removed net D2_P: U$4.B5
- removed net D4_N: U$4.A6
- removed net D4_P: U$4.B6
- removed net D5_N: U$4.E6
- removed net D5_P: U$4.F7
- removed net D7_N: U$4.C6
- removed net D7_P: U$4.D6
- removed net D8_N: U$4.A8
- removed net D8_P: U$4.B8
- removed net GP1: U$4.C4
- removed net GP2: U$4.A4
- removed net GP3: U$4.D5
- removed net GP4: U$4.C5
- removed net N$5: U$6.H1
- removed net N$6: U$6.M8
- removed net N$7: U$6.L8
- new net DDR_A15: U$2.M7
- new net DDR_DQM0: U$2.E7
- new net DDR_DQM1: U$2.D3
- new net DDR_DQS0_N: U$2.G3
- new net DDR_DQS0_P: U$2.F3
- new net DDR_DQS1_N: U$2.B7
- new net DDR_DQS1_P: U$2.C7
- new net DDR_UDQS: U$4.T15
- new net DDR_VERF: U$2.H1, U$2.M8
- new net N$12: U$4.K12
- new net N$13: U$4.K11
- new net N$22: U$4.N14
- new net N$23: U$4.N16
- new net N$3: R1.+, U$2.L8
- new net N$32: U$4.R14
- new net VCC_1.5: U$2.A1, U$2.A8, U$2.B2, U$2.C1, U$2.C9, U$2.D2, U$2.D9, U$2.E9, U$2.F1, U$2.G7, U$2.H2, U$2.H9, U$2.K2, U$2.K8, U$2.N1, U$2.N9, U$2.R1, U$2.R9
- net DDR_A0: now also U$2.N3; no longer U$6.N3
- net DDR_A1: now also U$2.P7; no longer U$6.P7
- net DDR_A10: now also U$2.L7; no longer U$6.L7
- net DDR_A11: now also U$2.R7; no longer U$6.R7
- net DDR_A12: now also U$2.N7; no longer U$6.N7
- net DDR_A13: now also U$2.T3; no longer U$6.T3
- net DDR_A14: now also U$2.T7; no longer U$6.T7
- net DDR_A2: now also U$2.P3; no longer U$6.P3
- net DDR_A3: now also U$2.N2, U$4.H13; no longer U$6.N2
- net DDR_A4: now also U$2.P8; no longer U$6.P8
- net DDR_A5: now also U$2.P2, U$4.J11; no longer U$6.P2
- net DDR_A6: now also U$2.R8, U$4.J12; no longer U$6.R8
- net DDR_A7: now also U$2.R2; no longer U$6.R2
- net DDR_A8: now also U$2.T8; no longer U$6.T8
- net DDR_A9: now also U$2.R3; no longer U$6.R3
- net DDR_BA0: now also U$2.M2; no longer U$6.M2
- net DDR_BA1: now also U$2.N8; no longer U$6.N8
- net DDR_BA2: now also U$2.M3; no longer U$6.M3
- net DDR_CAS: now also U$2.K3, U$4.K14; no longer U$6.K3
- net DDR_CKE: now also U$2.K9; no longer U$6.K9
- net DDR_CK_N: now also U$2.K7, U$4.H11; no longer U$6.K7
- net DDR_CK_P: now also U$2.J7, U$4.G12; no longer U$6.J7
- net DDR_CS: now also U$2.L2; no longer U$6.L2
- net DDR_DQ0: now also U$2.E3, U$4.L14; no longer U$6.E3
- net DDR_DQ1: now also U$2.F7, U$4.L16; no longer U$6.F7
- net DDR_DQ10: now also U$2.C8, U$4.R15; no longer U$6.C8
- net DDR_DQ11: now also U$2.C2, U$4.R16; no longer U$6.C2
- net DDR_DQ12: now also U$2.A7, U$4.T14; no longer U$6.A7
- net DDR_DQ13: now also U$2.A2, U$4.T13; no longer U$6.A2
- net DDR_DQ14: now also U$2.B8, U$4.R12; no longer U$6.B8
- net DDR_DQ15: now also U$2.A3, U$4.T12; no longer U$6.A3
- net DDR_DQ2: now also U$2.F2, U$4.M15; no longer U$6.F2
- net DDR_DQ3: now also U$2.F8, U$4.M16; no longer U$6.F8
- net DDR_DQ4: now also U$2.H3, U$4.J14; no longer U$6.H3
- net DDR_DQ5: now also U$2.H8, U$4.J16; no longer U$6.H8
- net DDR_DQ6: now also U$2.G2, U$4.K15; no longer U$6.G2
- net DDR_DQ7: now also U$2.H7, U$4.K16; no longer U$6.H7
- net DDR_DQ8: now also U$2.D7, U$4.P15; no longer U$6.D7
- net DDR_DQ9: now also U$2.C3, U$4.P16; no longer U$6.C3
- net DDR_ODT: now also U$2.K1, U$4.H14; no longer U$6.K1
- net DDR_RAS: now also U$2.J3, U$4.J13; no longer U$6.J3
- net DDR_REST: now also U$2.T2; no longer U$6.T2
- net DDR_WE: now also U$2.L3; no longer U$6.L3
- net GND: now also R1.-, U$2.A9, U$2.B1, U$2.B3, U$2.B9, U$2.D1, U$2.D8, U$2.E1, U$2.E2, U$2.E8, U$2.F9, U$2.G1, U$2.G8, U$2.G9, U$2.J2, U$2.J8, U$2.M1, U$2.M9, U$2.P1, U$2.P9, U$2.T1, U$2.T9; no longer U$6.A9, U$6.B1, U$6.B3, U$6.B9, U$6.D1, U$6.D8, U$6.E1, U$6.E2, U$6.E8, U$6.F9, U$6.G1, U$6.G8, U$6.G9, U$6.J2, U$6.J8, U$6.M1, U$6.M9, U$6.P1, U$6.P9, U$6.T1, U$6.T9
- net VCC15: no longer U$6.A1, U$6.A8, U$6.B2, U$6.C1, U$6.C9, U$6.D2, U$6.D9, U$6.E9, U$6.F1, U$6.G7, U$6.H2, U$6.H9, U$6.K2, U$6.K8, U$6.N9, U$6.R9
Routing:
- net D7_P: track 23.6 -> 0.00 mm, vias 1 -> 0
- net D7_N: track 23.3 -> 0.00 mm, vias 1 -> 0
- net DDR_DQ13: track 0.00 -> 21.6 mm
- net GND: track 54.4 -> 36.5 mm, vias 44 -> 29
- net DDR_DQ12: track 0.00 -> 14.7 mm
- net DDR_CK_N: track 0.00 -> 14.3 mm, vias 0 -> 1
- net DDR_CK_P: track 0.00 -> 13.8 mm, vias 0 -> 1
- net VCC15: track 26.5 -> 13.4 mm, vias 21 -> 8
- net DDR_A13: track 14.5 -> 13.5 mm
- net GP3: track 0.71 -> 0.00 mm, vias 1 -> 0
- net D5_P: track 0.71 -> 0.00 mm, vias 1 -> 0
- net D5_N: track 0.71 -> 0.00 mm, vias 1 -> 0
- net B0_G7: track 0.71 -> 0.00 mm, vias 1 -> 0
