File: spartan6/hardware/dockerkit.sch (EAGLE design)
At the start: 6 parts

Commit message: 调整电路
Parts:
- removed U$6: DDR3, FPGA:DDR3
- added R1: 240, Resistors&Capacitors:RESISTOR0402
- added U$2: DDR3, IC_Memory:DDR3
- U$4: device FPGA:XC6SLX16 -> IC_FPGA:XC6SLX16
Connections:
- removed net B0_G5: U$4.C7
- removed net B0_G6: U$4.A7
- removed net B0_G7: U$4.C9
- removed net B0_G8: U$4.A9
- removed net D2_N: U$4.A5
- removed net D2_P: U$4.B5
- removed net D4_N: U$4.A6
- removed net D4_P: U$4.B6
- removed net D5_N: U$4.E6
- removed net D5_P: U$4.F7
- removed net D7_N: U$4.C6
- removed net D7_P: U$4.D6
- removed net D8_N: U$4.A8
- removed net D8_P: U$4.B8
- removed net GP1: U$4.C4
- removed net GP2: U$4.A4
- removed net GP3: U$4.D5
- removed net GP4: U$4.C5
- removed net N$5: U$6.VREFDQ
- removed net N$6: U$6.VREFCA
- removed net N$7: U$6.ZQ
- new net DDR_A15: U$2.A15
- new net DDR_DQM0: U$2.LDM
- new net DDR_DQM1: U$2.UDM
- new net DDR_DQS0_N: U$2.LDQS_N
- new net DDR_DQS0_P: U$2.LDQS_P
- new net DDR_DQS1_N: U$2.UDQS_N
- new net DDR_DQS1_P: U$2.UDQS_P
- new net DDR_UDQS: U$4.IO_L50N_M1UDQSN_1
- new net DDR_VERF: U$2.VREFCA, U$2.VREFDQ
- new net N$12: U$4.IO_L42P_GCLK7_M1UDM_1
- new net N$13: U$4.IO_L42N_GCLK6_TRDY1_M1LDM_1
- new net N$22: U$4.IO_L45P_A1_M1LDQS_1
- new net N$23: U$4.IO_L45N_A0_M1LQSN_1
- new net N$3: R1.1, U$2.ZQ
- new net N$32: U$4.IO_L50P_M1UDQS_1
- new net VCC_1.5: U$2.VDD1, U$2.VDD2, U$2.VDD3, U$2.VDD4, U$2.VDD5, U$2.VDD6, U$2.VDD7, U$2.VDD8, U$2.VDD9, U$2.VDDQ1, U$2.VDDQ2, U$2.VDDQ3, U$2.VDDQ4, U$2.VDDQ5, U$2.VDDQ6, U$2.VDDQ7, U$2.VDDQ8, U$2.VDDQ9
- net DDR_A0: now also U$2.A0; no longer U$6.A0
- net DDR_A1: now also U$2.A1; no longer U$6.A1
- net DDR_A10: now also U$2.A10/AP; no longer U$6.A10/AP
- net DDR_A11: now also U$2.A11; no longer U$6.A11
- net DDR_A12: now also U$2.A12/BC#; no longer U$6.A12/BC#
- net DDR_A13: now also U$2.A13; no longer U$6.A13
- net DDR_A14: now also U$2.A14; no longer U$6.A14
- net DDR_A2: now also U$2.A2; no longer U$6.A2
- net DDR_A3: now also U$2.A3, U$4.IO_L39P_M1A3_1; no longer U$6.A3
- net DDR_A4: now also U$2.A4; no longer U$6.A4
- net DDR_A5: now also U$2.A5, U$4.IO_L40P_GCLK11_M1A5_1; no longer U$6.A5
- net DDR_A6: now also U$2.A6, U$4.IO_L40N_GCLK10_M1A6_1; no longer U$6.A6
- net DDR_A7: now also U$2.A7; no longer U$6.A7
- net DDR_A8: now also U$2.A8; no longer U$6.A8
- net DDR_A9: now also U$2.A9; no longer U$6.A9
- net DDR_BA0: now also U$2.BA0; no longer U$6.BA0
- net DDR_BA1: now also U$2.BA1; no longer U$6.BA1
- net DDR_BA2: now also U$2.BA2; no longer U$6.BA2
- net DDR_CAS: now also U$2.CAS#, U$4.IO_L41N_GCLK8_M1CASN_1; no longer U$6.CAS#
- net DDR_CKE: now also U$2.CKE; no longer U$6.CKE
- net DDR_CK_N: now also U$2.CK#, U$4.IO_L38N_A4_M1CLKN_1; no longer U$6.CK#
- net DDR_CK_P: now also U$2.CK, U$4.IO_L38P_A5_M1CLKP_1; no longer U$6.CK
- net DDR_CS: now also U$2.CS#; no longer U$6.CS#
- net DDR_DQ0: now also U$2.DQ0, U$4.IO_L47P_FWE_B_M1DQ0_1; no longer U$6.DQ0
- net DDR_DQ1: now also U$2.DQ1, U$4.IO_L47N_LDC_M1DQ1_1; no longer U$6.DQ1
- net DDR_DQ10: now also U$2.DQ10, U$4.IO_L49P_M1DQ10_1; no longer U$6.DQ10
- net DDR_DQ11: now also U$2.DQ11, U$4.IO_L49N_M1DQ11_1; no longer U$6.DQ11
- net DDR_DQ12: now also U$2.DQ12, U$4.IO_L51P_M1DQ12_1; no longer U$6.DQ12
- net DDR_DQ13: now also U$2.DQ13, U$4.IO_L51N_M1DQ13_1; no longer U$6.DQ13
- net DDR_DQ14: now also U$2.DQ14, U$4.IO_L52P_M1DQ14_1; no longer U$6.DQ14
- net DDR_DQ15: now also U$2.DQ15, U$4.IO_L52N_M1DQ15_1; no longer U$6.DQ15
- net DDR_DQ2: now also U$2.DQ2, U$4.IO_L46P_FCS_B_M1DQ2_1; no longer U$6.DQ2
- net DDR_DQ3: now also U$2.DQ3, U$4.IO_L46N_FOE_B_M1DQ3_1; no longer U$6.DQ3
- net DDR_DQ4: now also U$2.DQ4, U$4.IO_L43P_GCLK5_M1DQ4_1; no longer U$6.DQ4
- net DDR_DQ5: now also U$2.DQ5, U$4.IO_L43N_GCLK4_M1DQ5_1; no longer U$6.DQ5
- net DDR_DQ6: now also U$2.DQ6, U$4.IO_L44P_A3_M1DQ6_1; no longer U$6.DQ6
- net DDR_DQ7: now also U$2.DQ7, U$4.IO_L44N_A2_M1DQ7_1; no longer U$6.DQ7
- net DDR_DQ8: now also U$2.DQ8, U$4.IO_L48P_HDC_M1DQ8_1; no longer U$6.DQ8
- net DDR_DQ9: now also U$2.DQ9, U$4.IO_L48N_M1DQ9_1; no longer U$6.DQ9
- net DDR_ODT: now also U$2.ODT, U$4.IO_L39N_M1ODT_1; no longer U$6.ODT
- net DDR_RAS: now also U$2.RAS#, U$4.IO_L41P_GCLK9_IRDY1_M1RASN_1; no longer U$6.RAS#
- net DDR_REST: now also U$2.RESET#; no longer U$6.RESET#
- net DDR_WE: now also U$2.WE#; no longer U$6.WE#
- net GND: now also R1.2, U$2.VSS1, U$2.VSS10, U$2.VSS11, U$2.VSS12, U$2.VSS2, U$2.VSS3, U$2.VSS4, U$2.VSS5, U$2.VSS6, U$2.VSS7, U$2.VSS8, U$2.VSS9, U$2.VSSQ1, U$2.VSSQ2, U$2.VSSQ3, U$2.VSSQ4, U$2.VSSQ5, U$2.VSSQ6, U$2.VSSQ7, U$2.VSSQ8, U$2.VSSQ9; no longer U$6.VSS, U$6.VSSQ
- net VCC15: no longer U$6.VDD, U$6.VDDQ
